Commit message: Update README.md, add lidar.xacro, and amcl_config.yaml, and modify robot_core.xacro and rsp.launch.py

File: src/kinisirobot/description/robot.urdf.xacro (robot description, xacro)
@@ -2,3 +2,4 @@
 <robot xmlns:xacro="http://www.ros.org/wiki/xacro" name="robot">
     <xacro:include filename="robot_core.xacro"/>
+    <xacro:include filename="lidar.xacro"/>
 </robot>

File: src/kinisirobot/description/robot_core.xacro (robot description, xacro)
@@ -7,32 +7,17 @@
         <color rgba="0 0 0 1"/>
     </material>
-    <link name="base_link">
-    </link>
+    <link name="base_link"></link>
     <joint name="chassis_joint" type="fixed">
         <parent link="base_link"/>
         <child link="chassis"/>
-        <origin xyz="-0.1 0 0"/>
+        <origin xyz="0 0 0.05"/>
     </joint>
     <link name="chassis">
         <visual>
             <geometry>
-                <box size="0.3 0.3 0.15"/>
+                <cylinder radius="0.30" length="0.1"/>
             </geometry>
             <material name="white"/>
         </visual>
     </link>
-    <joint name="first_wheel_joint" type="continuous">
-        <parent link="chassis"/>
-        <child link="first_wheel"/>
-        <origin xyz="0.15 0 0" rpy="-${pi/2} 0 0"/>
-        <axis xyz="0 0 1"/>
-    </joint>
-    <link name="first_wheel">
-        <visual>
-            <geometry>
-                <cylinder radius="0.05" length="0.1"/>
-            </geometry>
-            <material name="black"/>
-        </visual>
-    </link>
 </robot>
