Commit message: Update robot parameters

File: src/kinisirobot/description/lidar.xacro (robot description, xacro)
@@ -7,5 +7,5 @@
         <parent link="chassis"/>
         <child link="laser_frame"/>
-        <origin xyz="0.1 0.0 0.075" rpy="0 0 0"/>
+        <origin xyz="0.115 0.0 0.075" rpy="0 0 0"/>
     </joint>
     <link name="laser_frame">

Commit message: Update lidar.xacro to rotate laser_joint by 180 degrees

File: src/kinisirobot/description/lidar.xacro (robot description, xacro)
@@ -7,5 +7,5 @@
         <parent link="chassis"/>
         <child link="laser_frame"/>
-        <origin xyz="0.115 0.0 0.075" rpy="0 0 0"/>
+        <origin xyz="0.115 0.0 0.075" rpy="0 0 3.14159"/>
     </joint>
     <link name="laser_frame">

Commit message: fix lidar pose

File: src/kinisirobot/description/lidar.xacro (robot description, xacro)
@@ -7,5 +7,5 @@
         <parent link="chassis"/>
         <child link="laser_frame"/>
-        <origin xyz="0.115 0.0 0.075" rpy="0 0 3.14159"/>
+        <origin xyz="0.115 0.0 0.075" rpy="0 0 0"/>
     </joint>
     <link name="laser_frame">

Commit message: Fix

File: src/kinisirobot/description/lidar.xacro (robot description, xacro)
@@ -7,5 +7,5 @@
         <parent link="chassis"/>
         <child link="laser_frame"/>
-        <origin xyz="0.115 0.0 0.075" rpy="0 0 0"/>
+        <origin xyz="0.115 0.0 0.075" rpy="3.14 0 0"/>
     </joint>
     <link name="laser_frame">

Commit message: Update robot parameters

File: src/kinisirobot/description/lidar.xacro (robot description, xacro)
@@ -7,5 +7,5 @@
         <parent link="chassis"/>
         <child link="laser_frame"/>
-        <origin xyz="0.115 0.0 0.075" rpy="3.14 0 0"/>
+        <origin xyz="0.112 0.0 0.075" rpy="0 3.14 0"/>
     </joint>
     <link name="laser_frame">

Commit message: update

File: src/kinisirobot/description/lidar.xacro (robot description, xacro)
@@ -7,5 +7,5 @@
         <parent link="chassis"/>
         <child link="laser_frame"/>
-        <origin xyz="0.112 0.0 0.075" rpy="0 3.14 0"/>
+        <origin xyz="0.112 0.0 0.075" rpy="3.14 0 3.14"/>
     </joint>
     <link name="laser_frame">

Commit message: fix

File: src/kinisirobot/description/lidar.xacro (robot description, xacro)
@@ -7,5 +7,5 @@
         <parent link="chassis"/>
         <child link="laser_frame"/>
-        <origin xyz="0.112 0.0 0.075" rpy="3.14 0 3.14"/>
+        <origin xyz="0.112 0.0 0.075" rpy="0 0 3.14"/>
     </joint>
     <link name="laser_frame">

Commit message: fix

File: src/kinisirobot/description/lidar.xacro (robot description, xacro)
@@ -7,5 +7,5 @@
         <parent link="chassis"/>
         <child link="laser_frame"/>
-        <origin xyz="0.112 0.0 0.075" rpy="0 0 3.14"/>
+        <origin xyz="0.112 0.0 0.075" rpy="0 0 0"/>
     </joint>
     <link name="laser_frame">

Commit message: fix

File: src/kinisirobot/description/lidar.xacro (robot description, xacro)
@@ -7,5 +7,5 @@
         <parent link="chassis"/>
         <child link="laser_frame"/>
-        <origin xyz="0.112 0.0 0.075" rpy="0 0 0"/>
+        <origin xyz="0.112 0.0 0.075" rpy="0 0 3.14"/>
     </joint>
     <link name="laser_frame">
