Commit message: Update omni navigation and odometry; add robot web client

File: src/kinisirobot/description/lidar.xacro (robot description, xacro)
@@ -7,5 +7,6 @@
         <parent link="chassis"/>
         <child link="laser_frame"/>
-        <origin xyz="0.115 0.0 0.075" rpy="0 0 0"/>
+        <!-- yaw=pi: RPLIDAR mounted rotated 180deg about Z (0deg beam faces rear). -->
+        <origin xyz="0.115 0.0 0.075" rpy="0 0 3.14159"/>
     </joint>
     <link name="laser_frame">
